File: gonk.sch (KiCad schematic (older format))
At the start: 4 parts, among them J1 AudioJack4, J2 AudioJack4, U1 ProMicro, U2 ProMicro

Commit message: 3D render checked
Parts:
- removed J1, J2: AudioJack4, symbol Connector:AudioJack4
- removed U1, U2: ProMicro, symbol promicro:ProMicro
- added J1: Conn_01x04_Female, Connector_PinSocket_2.54mm:PinSocket_1x04_P2.54mm_Vertical, symbol Connector:Conn_01x04_Female
- added U3, U4: kb2040, kb2040:kb2040, symbol gonk:kb2040
Connections:
- net GND: now also J1.1 (Pin_1), U4.16 (GND)
- net col0_L: now also U4.9 (D5)
- net col0_R: now also U3.9 (D5)
- net col1_L: now also U4.10 (D6)
- net col1_R: now also U3.10 (D6)
- net col2_L: now also U4.11 (D7)
- net col2_R: now also U3.11 (D7)
- net col3_L: now also U4.12 (D8)
- net col3_R: now also U3.12 (D8)
- net col4_L: now also U4.13 (D9)
- net col4_R: now also U3.13 (D9)
- net col5_L: now also U4.19 (A3)
- net col5_R: now also U3.19 (A3)
- net col6_L: now also U4.20 (A2)
- net col6_R: now also U3.20 (A2)
- net row0_L: now also U4.2 (D0)
- net row0_R: now also U3.2 (D0)
- net row1_L: now also U4.3 (D1)
- net row1_R: now also U3.3 (D1)
- net row2_L: now also U4.6 (D2)
- net row2_R: now also U3.21 (A1)
- net row3_L: now also U4.7 (D3)
- net row3_R: now also U3.22 (A0)
- net row4_L: now also U4.8 (D4)
- net row4_R: now also U3.8 (D4)
- new net RAW: J1.2 (Pin_2), U4.15 (RAW)
- new net SCL: J1.3 (Pin_3), U3.7 (D3)
- new net SDA: J1.4 (Pin_4), U3.6 (D2)
Other:
- note added: "5V\n500 mA to 1A\n"
- note added: "Features:\n- KB2040 with castellated pins\n- Split with TRRS connection\n- Blueooth X\n- USB C \n- Switchable OLED"
- note removed: "Features:\n- Split with TRRS connection\n- Blueooth X\n- USB C \n- Switchable OLED"
Changed lines of the file:
@@
 Comment4 ""
 $EndDescr
-Text Notes 10000 950  0    50   ~ 0
-Features:\n- Split with TRRS connection\n- Blueooth X\n- USB C \n- Switchable OLED
-Text GLabel 1250 5650 2    50   Input ~ 0
-data
-Text GLabel 2450 5650 2    50   Input ~ 0
-data
-$Comp
-L power:VCC #PWR0102
-U 1 1 61C47311
-P 1250 5450
-F 0 "#PWR0102" H 1250 5300 50  0001 C CNN
-F 1 "VCC" V 1265 5578 50  0000 L CNN
-F 2 "" H 1250 5450 50  0001 C CNN
-F 3 "" H 1250 5450 50  0001 C CNN
-	1    1250 5450
-	0    1    1    0
-$EndComp
-$Comp
-L power:VCC #PWR0103
-U 1 1 61C48084
-P 2450 5450
-F 0 "#PWR0103" H 2450 5300 50  0001 C CNN
-F 1 "VCC" V 2465 5578 50  0000 L CNN
-F 2 "" H 2450 5450 50  0001 C CNN
-F 3 "" H 2450 5450 50  0001 C CNN
-	1    2450 5450
-	0    1    1    0
-$EndComp
-$Comp
-L power:GND #PWR0104
-U 1 1 61C486D1
-P 1250 5550
-F 0 "#PWR0104" H 1250 5300 50  0001 C CNN
-F 1 "GND" V 1255 5422 50  0000 R CNN
-F 2 "" H 1250 5550 50  0001 C CNN
-F 3 "" H 1250 5550 50  0001 C CNN
-	1    1250 5550
-	0    -1   -1   0
-$EndComp
-$Comp
-L power:GND #PWR0105
-U 1 1 61C48EE4
-P 2450 5550
-F 0 "#PWR0105" H 2450 5300 50  0001 C CNN
-F 1 "GND" V 2455 5422 50  0000 R CNN
-F 2 "" H 2450 5550 50  0001 C CNN
-F 3 "" H 2450 5550 50  0001 C CNN
-	1    2450 5550
-	0    -1   -1   0
-$EndComp
+Text Notes 9950 1000 0    50   ~ 0
+Features:\n- KB2040 with castellated pins\n- Split with TRRS connection\n- Blueooth X\n- USB C \n- Switchable OLED
 $Sheet
 S 800  700  1650 1300
@@
 F9 "col5" I R 2450 1300 50
 F10 "col6" I R 2450 1400 50
-F12 "row2" I L 800 1000 50
-F13 "row3" I L 800 1100 50
-F14 "row4" I L 800 1200 50
+F11 "row2" I L 800 1000 50
+F12 "row3" I L 800 1100 50
+F13 "row4" I L 800 1200 50
 $EndSheet
 Text Notes 500  600  0    50   ~ 0
@@
 Text Label 800  800  2    50   ~ 0
 row0_L
-$Comp
-L Connector:AudioJack4 J1
-U 1 1 61C79B69
-P 1050 5450
-F 0 "J1" H 1007 5775 50  0000 C CNN
-F 1 "AudioJack4" H 1007 5684 50  0000 C CNN
-F 2 "" H 1050 5450 50  0001 C CNN
-F 3 "~" H 1050 5450 50  0001 C CNN
-	1    1050 5450
-	1    0    0    -1
-$EndComp
-$Comp
-L Connector:AudioJack4 J2
-U 1 1 61C7B0C6
-P 2250 5450
-F 0 "J2" H 2207 5775 50  0000 C CNN
-F 1 "AudioJack4" H 2207 5684 50  0000 C CNN
-F 2 "" H 2250 5450 50  0001 C CNN
-F 3 "~" H 2250 5450 50  0001 C CNN
-	1    2250 5450
-	1    0    0    -1
-$EndComp
-$Comp
-L promicro:ProMicro U1
-U 1 1 61D3394E
-P 4300 1600
-F 0 "U1" H 4300 2637 60  0000 C CNN
-F 1 "ProMicro" H 4300 2531 60  0000 C CNN
-F 2 "" H 4400 550 60  0000 C CNN
-F 3 "" H 4400 550 60  0000 C CNN
-	1    4300 1600
-	1    0    0    -1
-$EndComp
-$Comp
-L promicro:ProMicro U2
-U 1 1 61CA32E6
-P 4400 3500
-F 0 "U2" H 4400 4537 60  0000 C CNN
-F 1 "ProMicro" H 4400 4431 60  0000 C CNN
-F 2 "" H 4500 2450 60  0000 C CNN
-F 3 "" H 4500 2450 60  0000 C CNN
-	1    4400 3500
-	1    0    0    -1
-$EndComp
 Text Label 800  900  2    50   ~ 0
 row1_L
@@
 F9 "col5" I R 2550 3200 50
 F10 "col6" I R 2550 3300 50
-F12 "row2" I L 900 2900 50
-F13 "row3" I L 900 3000 50
-F14 "row4" I L 900 3100 50
+F11 "row2" I L 900 2900 50
+F12 "row3" I L 900 3000 50
+F13 "row4" I L 900 3100 50
 $EndSheet
 Text Label 900  2700 2    50   ~ 0
@@
 Wire Notes Line
 	6300 500  6300 4150
-Text Label 3600 1450 2    50   ~ 0
+Text Label 3650 850  2    50   ~ 0
 row0_L
-Text Label 3600 1550 2    50   ~ 0
+Text Label 3650 950  2    50   ~ 0
 row1_L
-Text Label 3600 1650 2    50   ~ 0
+Text Label 3650 1250 2    50   ~ 0
 row2_L
-Text Label 3600 1750 2    50   ~ 0
+Text Label 3650 1350 2    50   ~ 0
 row3_L
-Text Label 3600 1850 2    50   ~ 0
+Text Label 3650 1450 2    50   ~ 0
 row4_L
-Text Label 3600 1950 2    50   ~ 0
+Text Label 3650 1550 2    50   ~ 0
 col0_L
-Text Label 5000 1250 0    50   ~ 0
+Text Label 3650 1650 2    50   ~ 0
 col1_L
 Text Label 2450 1000 0    50   ~ 0
 col2_L
-Text Label 5000 1350 0    50   ~ 0
+Text Label 3650 1750 2    50   ~ 0
 col2_L
-Text Label 5000 1450 0    50   ~ 0
+Text Label 3650 1850 2    50   ~ 0
 col3_L
-Text Label 5000 1550 0    50   ~ 0
+Text Label 3650 1950 2    50   ~ 0
 col4_L
-Text Label 5000 1650 0    50   ~ 0
+Text Label 4250 1250 0    50   ~ 0
 col5_L
-Text Label 5000 1750 0    50   ~ 0
+Text Label 4250 1350 0    50   ~ 0
 col6_L
-Text Label 3700 3350 2    50   ~ 0
+Text Label 3650 2850 2    50   ~ 0
 row0_R
-Text Label 3700 3450 2    50   ~ 0
+Text Label 3650 2950 2    50   ~ 0
 row1_R
-Text Label 3700 3550 2    50   ~ 0
+Text Label 4250 3450 0    50   ~ 0
 row2_R
-Text Label 3700 3650 2    50   ~ 0
+Text Label 4250 3550 0    50   ~ 0
 row3_R
-Text Label 3700 3750 2    50   ~ 0
+Text Label 3650 3450 2    50   ~ 0
 row4_R
-Text Label 3700 3850 2    50   ~ 0
+Text Label 3650 3550 2    50   ~ 0
 col0_R
-Text Label 5100 3150 0    50   ~ 0
+Text Label 4250 3250 0    50   ~ 0
+col5_R
+Text Label 4250 3350 0    50   ~ 0
+col6_R
+$Comp
+L Connector:Conn_01x04_Female J1
+U 1 1 61CF838B
+P 7250 700
+F 0 "J1" H 7278 676 50  0000 L CNN
+F 1 "Conn_01x04_Female" H 7278 585 50  0000 L CNN
+F 2 "Connector_PinSocket_2.54mm:PinSocket_1x04_P2.54mm_Vertical" H 7250 700 50  0001 C CNN
+F 3 "~" H 7250 700 50  0001 C CNN
+	1    7250 700
+	1    0    0    -1
+$EndComp
+$Comp
+L power:GND #PWR0103
+U 1 1 61CFE11C
+P 4250 950
+F 0 "#PWR0103" H 4250 700 50  0001 C CNN
+F 1 "GND" V 4255 822 50  0000 R CNN
+F 2 "" H 4250 950 50  0001 C CNN
+F 3 "" H 4250 950 50  0001 C CNN
+	1    4250 950
+	0    -1   -1   0
+$EndComp
+$Comp
+L power:GND #PWR0107
+U 1 1 61CFFC79
+P 7050 600
+F 0 "#PWR0107" H 7050 350 50  0001 C CNN
+F 1 "GND" V 7055 472 50  0000 R CNN
+F 2 "" H 7050 600 50  0001 C CNN
+F 3 "" H 7050 600 50  0001 C CNN
+	1    7050 600
+	0    1    1    0
+$EndComp
+Text Label 3650 3350 2    50   ~ 0
+SCL
+Text Label 3650 3250 2    50   ~ 0
+SDA
+Text Label 7050 800  2    50   ~ 0
+SCL
+Text Label 7050 900  2    50   ~ 0
+SDA
+Text Label 4250 850  0    50   ~ 0
+RAW
+Text Label 7050 700  2    50   ~ 0
+RAW
+Text Notes 4450 850  0    50   ~ 0
+5V\n500 mA to  1A\n
+$Comp
+L gonk:kb2040 U4
+U 1 1 61D0D424
+P 3950 1150
+F 0 "U4" H 3950 1815 50  0000 C CNN
+F 1 "kb2040" H 3950 1724 50  0000 C CNN
+F 2 "kb2040:kb2040" H 3950 1150 50  0001 C CNN
+F 3 "" H 3950 1150 50  0001 C CNN
+	1    3950 1150
+	1    0    0    -1
+$EndComp
+$Comp
+L gonk:kb2040 U3
+U 1 1 61D12A11
+P 3950 3150
+F 0 "U3" H 3950 3815 50  0000 C CNN
+F 1 "kb2040" H 3950 3724 50  0000 C CNN
+F 2 "kb2040:kb2040" H 3950 3150 50  0001 C CNN
+F 3 "" H 3950 3150 50  0001 C CNN
+	1    3950 3150
+	1    0    0    -1
+$EndComp
+Text Label 3650 3950 2    50   ~ 0
+col4_R
+Text Label 3650 3850 2    50   ~ 0
+col3_R
+Text Label 3650 3750 2    50   ~ 0
+col2_R
+Text Label 3650 3650 2    50   ~ 0
 col1_R
-Text Label 5100 3250 0    50   ~ 0
-col2_R
-Text Label 5100 3350 0    50   ~ 0
-col3_R
-Text Label 5100 3450 0    50   ~ 0
-col4_R
-Text Label 5100 3550 0    50   ~ 0
-col5_R
-Text Label 5100 3650 0    50   ~ 0
-col6_R
 $EndSCHEMATC
