File: key_array.sch (KiCad schematic (older format))
At the start: 70 parts, among them K1 KEYSW, K10 KEYSW, K11 KEYSW, K12 KEYSW, K13 KEYSW, K14 KEYSW, K15 KEYSW, K16 KEYSW, K17 KEYSW, K18 KEYSW, K19 KEYSW, K2 KEYSW, K20 KEYSW, K21 KEYSW, K22 KEYSW, K23 KEYSW, K24 KEYSW, K25 KEYSW, K26 KEYSW, K27 KEYSW, K28 KEYSW, K29 KEYSW, K3 KEYSW, K30 KEYSW, K31 KEYSW, K32 KEYSW, K33 KEYSW, K34 KEYSW, K35 KEYSW, K4 KEYSW, K5 KEYSW, K6 KEYSW, K7 KEYSW, K8 KEYSW, K9 KEYSW

Commit message: 3D render checked
Parts:
- K1, K10, K11, K12, K13, K14, K15, K16, K17, K18, K19, K2, K20, K21, K22, K23, K24, K25, K26, K27, K28, K29, K3, K30, K31, K32, K33, K34, K35, K4, K5, K6, K7, K8, K9: footprint keyswitches:SW_PG1350 -> gonk_footprint:Kailh_socket_PG1350
Changed lines of the file:
@@
 F 0 "K6" H 4150 4033 60  0000 C CNN
 F 1 "KEYSW" H 4150 3700 60  0001 C CNN
-F 2 "keyswitches:SW_PG1350" H 4150 3800 60  0001 C CNN
+F 2 "gonk_footprint:Kailh_socket_PG1350" H 4150 3800 60  0001 C CNN
 F 3 "" H 4150 3800 60  0000 C CNN
 	1    4150 3800
@@
 F 0 "K5" H 4150 3383 60  0000 C CNN
 F 1 "KEYSW" H 4150 3050 60  0001 C CNN
-F 2 "keyswitches:SW_PG1350" H 4150 3150 60  0001 C CNN
+F 2 "gonk_footprint:Kailh_socket_PG1350" H 4150 3150 60  0001 C CNN
 F 3 "" H 4150 3150 60  0000 C CNN
 	1    4150 3150
@@
 F 0 "K2" H 3200 4033 60  0000 C CNN
 F 1 "KEYSW" H 3200 3700 60  0001 C CNN
-F 2 "keyswitches:SW_PG1350" H 3200 3800 60  0001 C CNN
+F 2 "gonk_footprint:Kailh_socket_PG1350" H 3200 3800 60  0001 C CNN
 F 3 "" H 3200 3800 60  0000 C CNN
 	1    3200 3800
@@
 F 0 "K1" H 3200 3383 60  0000 C CNN
 F 1 "KEYSW" H 3200 3050 60  0001 C CNN
-F 2 "keyswitches:SW_PG1350" H 3200 3150 60  0001 C CNN
+F 2 "gonk_footprint:Kailh_socket_PG1350" H 3200 3150 60  0001 C CNN
 F 3 "" H 3200 3150 60  0000 C CNN
 	1    3200 3150
@@
 F 0 "K14" H 6100 4033 60  0000 C CNN
 F 1 "KEYSW" H 6100 3700 60  0001 C CNN
-F 2 "keyswitches:SW_PG1350" H 6100 3800 60  0001 C CNN
+F 2 "gonk_footprint:Kailh_socket_PG1350" H 6100 3800 60  0001 C CNN
 F 3 "" H 6100 3800 60  0000 C CNN
 	1    6100 3800
@@
 F 0 "K13" H 6100 3383 60  0000 C CNN
 F 1 "KEYSW" H 6100 3050 60  0001 C CNN
-F 2 "keyswitches:SW_PG1350" H 6100 3150 60  0001 C CNN
+F 2 "gonk_footprint:Kailh_socket_PG1350" H 6100 3150 60  0001 C CNN
 F 3 "" H 6100 3150 60  0000 C CNN
 	1    6100 3150
@@
 F 0 "K10" H 5150 4033 60  0000 C CNN
 F 1 "KEYSW" H 5150 3700 60  0001 C CNN
-F 2 "keyswitches:SW_PG1350" H 5150 3800 60  0001 C CNN
+F 2 "gonk_footprint:Kailh_socket_PG1350" H 5150 3800 60  0001 C CNN
 F 3 "" H 5150 3800 60  0000 C CNN
 	1    5150 3800
@@
 F 0 "K9" H 5150 3383 60  0000 C CNN
 F 1 "KEYSW" H 5150 3050 60  0001 C CNN
-F 2 "keyswitches:SW_PG1350" H 5150 3150 60  0001 C CNN
+F 2 "gonk_footprint:Kailh_socket_PG1350" H 5150 3150 60  0001 C CNN
 F 3 "" H 5150 3150 60  0000 C CNN
 	1    5150 3150
@@
 F 0 "K22" H 8100 4033 60  0000 C CNN
 F 1 "KEYSW" H 8100 3700 60  0001 C CNN
-F 2 "keyswitches:SW_PG1350" H 8100 3800 60  0001 C CNN
+F 2 "gonk_footprint:Kailh_socket_PG1350" H 8100 3800 60  0001 C CNN
 F 3 "" H 8100 3800 60  0000 C CNN
 	1    8100 3800
@@
 F 0 "K21" H 8100 3383 60  0000 C CNN
 F 1 "KEYSW" H 8100 3050 60  0001 C CNN
-F 2 "keyswitches:SW_PG1350" H 8100 3150 60  0001 C CNN
+F 2 "gonk_footprint:Kailh_socket_PG1350" H 8100 3150 60  0001 C CNN
 F 3 "" H 8100 3150 60  0000 C CNN
 	1    8100 3150
@@
 F 0 "K18" H 7150 4033 60  0000 C CNN
 F 1 "KEYSW" H 7150 3700 60  0001 C CNN
-F 2 "keyswitches:SW_PG1350" H 7150 3800 60  0001 C CNN
+F 2 "gonk_footprint:Kailh_socket_PG1350" H 7150 3800 60  0001 C CNN
 F 3 "" H 7150 3800 60  0000 C CNN
 	1    7150 3800
@@
 F 0 "K17" H 7150 3383 60  0000 C CNN
 F 1 "KEYSW" H 7150 3050 60  0001 C CNN
-F 2 "keyswitches:SW_PG1350" H 7150 3150 60  0001 C CNN
+F 2 "gonk_footprint:Kailh_socket_PG1350" H 7150 3150 60  0001 C CNN
 F 3 "" H 7150 3150 60  0000 C CNN
 	1    7150 3150
@@
 F 0 "K26" H 9100 4033 60  0000 C CNN
 F 1 "KEYSW" H 9100 3700 60  0001 C CNN
-F 2 "keyswitches:SW_PG1350" H 9100 3800 60  0001 C CNN
+F 2 "gonk_footprint:Kailh_socket_PG1350" H 9100 3800 60  0001 C CNN
 F 3 "" H 9100 3800 60  0000 C CNN
 	1    9100 3800
@@
 F 0 "K25" H 9100 3383 60  0000 C CNN
 F 1 "KEYSW" H 9100 3050 60  0001 C CNN
-F 2 "keyswitches:SW_PG1350" H 9100 3150 60  0001 C CNN
+F 2 "gonk_footprint:Kailh_socket_PG1350" H 9100 3150 60  0001 C CNN
 F 3 "" H 9100 3150 60  0000 C CNN
 	1    9100 3150
@@
 F 0 "K8" H 4150 5333 60  0000 C CNN
 F 1 "KEYSW" H 4150 5000 60  0001 C CNN
-F 2 "keyswitches:SW_PG1350" H 4150 5100 60  0001 C CNN
+F 2 "gonk_footprint:Kailh_socket_PG1350" H 4150 5100 60  0001 C CNN
 F 3 "" H 4150 5100 60  0000 C CNN
 	1    4150 5100
@@
 F 0 "K7" H 4150 4683 60  0000 C CNN
 F 1 "KEYSW" H 4150 4350 60  0001 C CNN
-F 2 "keyswitches:SW_PG1350" H 4150 4450 60  0001 C CNN
+F 2 "gonk_footprint:Kailh_socket_PG1350" H 4150 4450 60  0001 C CNN
 F 3 "" H 4150 4450 60  0000 C CNN
 	1    4150 4450
@@
 F 0 "K4" H 3200 5333 60  0000 C CNN
 F 1 "KEYSW" H 3200 5000 60  0001 C CNN
-F 2 "keyswitches:SW_PG1350" H 3200 5100 60  0001 C CNN
+F 2 "gonk_footprint:Kailh_socket_PG1350" H 3200 5100 60  0001 C CNN
 F 3 "" H 3200 5100 60  0000 C CNN
 	1    3200 5100
@@
 F 0 "K3" H 3200 4683 60  0000 C CNN
 F 1 "KEYSW" H 3200 4350 60  0001 C CNN
-F 2 "keyswitches:SW_PG1350" H 3200 4450 60  0001 C CNN
+F 2 "gonk_footprint:Kailh_socket_PG1350" H 3200 4450 60  0001 C CNN
 F 3 "" H 3200 4450 60  0000 C CNN
 	1    3200 4450
@@
 F 0 "K16" H 6100 5333 60  0000 C CNN
 F 1 "KEYSW" H 6100 5000 60  0001 C CNN
-F 2 "keyswitches:SW_PG1350" H 6100 5100 60  0001 C CNN
+F 2 "gonk_footprint:Kailh_socket_PG1350" H 6100 5100 60  0001 C CNN
 F 3 "" H 6100 5100 60  0000 C CNN
 	1    6100 5100
@@
 F 0 "K15" H 6100 4683 60  0000 C CNN
 F 1 "KEYSW" H 6100 4350 60  0001 C CNN
-F 2 "keyswitches:SW_PG1350" H 6100 4450 60  0001 C CNN
+F 2 "gonk_footprint:Kailh_socket_PG1350" H 6100 4450 60  0001 C CNN
 F 3 "" H 6100 4450 60  0000 C CNN
 	1    6100 4450
@@
 F 0 "K12" H 5150 5333 60  0000 C CNN
 F 1 "KEYSW" H 5150 5000 60  0001 C CNN
-F 2 "keyswitches:SW_PG1350" H 5150 5100 60  0001 C CNN
+F 2 "gonk_footprint:Kailh_socket_PG1350" H 5150 5100 60  0001 C CNN
 F 3 "" H 5150 5100 60  0000 C CNN
 	1    5150 5100
@@
 F 0 "K24" H 8100 5333 60  0000 C CNN
 F 1 "KEYSW" H 8100 5000 60  0001 C CNN
-F 2 "keyswitches:SW_PG1350" H 8100 5100 60  0001 C CNN
+F 2 "gonk_footprint:Kailh_socket_PG1350" H 8100 5100 60  0001 C CNN
 F 3 "" H 8100 5100 60  0000 C CNN
 	1    8100 5100
@@
 F 0 "K23" H 8100 4683 60  0000 C CNN
 F 1 "KEYSW" H 8100 4350 60  0001 C CNN
-F 2 "keyswitches:SW_PG1350" H 8100 4450 60  0001 C CNN
+F 2 "gonk_footprint:Kailh_socket_PG1350" H 8100 4450 60  0001 C CNN
 F 3 "" H 8100 4450 60  0000 C CNN
 	1    8100 4450
@@
 F 0 "K20" H 7150 5333 60  0000 C CNN
 F 1 "KEYSW" H 7150 5000 60  0001 C CNN
-F 2 "keyswitches:SW_PG1350" H 7150 5100 60  0001 C CNN
+F 2 "gonk_footprint:Kailh_socket_PG1350" H 7150 5100 60  0001 C CNN
 F 3 "" H 7150 5100 60  0000 C CNN
 	1    7150 5100
@@
 F 0 "K19" H 7150 4683 60  0000 C CNN
 F 1 "KEYSW" H 7150 4350 60  0001 C CNN
-F 2 "keyswitches:SW_PG1350" H 7150 4450 60  0001 C CNN
+F 2 "gonk_footprint:Kailh_socket_PG1350" H 7150 4450 60  0001 C CNN
 F 3 "" H 7150 4450 60  0000 C CNN
 	1    7150 4450
@@
 F 0 "K28" H 9100 5333 60  0000 C CNN
 F 1 "KEYSW" H 9100 5000 60  0001 C CNN
-F 2 "keyswitches:SW_PG1350" H 9100 5100 60  0001 C CNN
+F 2 "gonk_footprint:Kailh_socket_PG1350" H 9100 5100 60  0001 C CNN
 F 3 "" H 9100 5100 60  0000 C CNN
 	1    9100 5100
@@
 F 0 "K27" H 9100 4683 60  0000 C CNN
 F 1 "KEYSW" H 9100 4350 60  0001 C CNN
-F 2 "keyswitches:SW_PG1350" H 9100 4450 60  0001 C CNN
+F 2 "gonk_footprint:Kailh_socket_PG1350" H 9100 4450 60  0001 C CNN
 F 3 "" H 9100 4450 60  0000 C CNN
 	1    9100 4450
@@
 F 0 "K11" H 5150 4683 60  0000 C CNN
 F 1 "KEYSW" H 5150 4350 60  0001 C CNN
-F 2 "keyswitches:SW_PG1350" H 5150 4450 60  0001 C CNN
+F 2 "gonk_footprint:Kailh_socket_PG1350" H 5150 4450 60  0001 C CNN
 F 3 "" H 5150 4450 60  0000 C CNN
 	1    5150 4450
@@
 F 0 "K30" H 4150 5983 60  0000 C CNN
 F 1 "KEYSW" H 4150 5650 60  0001 C CNN
-F 2 "keyswitches:SW_PG1350" H 4150 5750 60  0001 C CNN
+F 2 "gonk_footprint:Kailh_socket_PG1350" H 4150 5750 60  0001 C CNN
 F 3 "" H 4150 5750 60  0000 C CNN
 	1    4150 5750
@@
 F 0 "K29" H 3200 5983 60  0000 C CNN
 F 1 "KEYSW" H 3200 5650 60  0001 C CNN
-F 2 "keyswitches:SW_PG1350" H 3200 5750 60  0001 C CNN
+F 2 "gonk_footprint:Kailh_socket_PG1350" H 3200 5750 60  0001 C CNN
 F 3 "" H 3200 5750 60  0000 C CNN
 	1    3200 5750
@@
 F 0 "K32" H 6100 5983 60  0000 C CNN
 F 1 "KEYSW" H 6100 5650 60  0001 C CNN
-F 2 "keyswitches:SW_PG1350" H 6100 5750 60  0001 C CNN
+F 2 "gonk_footprint:Kailh_socket_PG1350" H 6100 5750 60  0001 C CNN
 F 3 "" H 6100 5750 60  0000 C CNN
 	1    6100 5750
@@
 F 0 "K31" H 5150 5983 60  0000 C CNN
 F 1 "KEYSW" H 5150 5650 60  0001 C CNN
-F 2 "keyswitches:SW_PG1350" H 5150 5750 60  0001 C CNN
+F 2 "gonk_footprint:Kailh_socket_PG1350" H 5150 5750 60  0001 C CNN
 F 3 "" H 5150 5750 60  0000 C CNN
 	1    5150 5750
@@
 F 0 "K34" H 8100 5983 60  0000 C CNN
 F 1 "KEYSW" H 8100 5650 60  0001 C CNN
-F 2 "keyswitches:SW_PG1350" H 8100 5750 60  0001 C CNN
+F 2 "gonk_footprint:Kailh_socket_PG1350" H 8100 5750 60  0001 C CNN
 F 3 "" H 8100 5750 60  0000 C CNN
 	1    8100 5750
@@
 F 0 "K33" H 7150 5983 60  0000 C CNN
 F 1 "KEYSW" H 7150 5650 60  0001 C CNN
-F 2 "keyswitches:SW_PG1350" H 7150 5750 60  0001 C CNN
+F 2 "gonk_footprint:Kailh_socket_PG1350" H 7150 5750 60  0001 C CNN
 F 3 "" H 7150 5750 60  0000 C CNN
 	1    7150 5750
@@
 F 0 "K35" H 9100 5983 60  0000 C CNN
 F 1 "KEYSW" H 9100 5650 60  0001 C CNN
-F 2 "keyswitches:SW_PG1350" H 9100 5750 60  0001 C CNN
+F 2 "gonk_footprint:Kailh_socket_PG1350" H 9100 5750 60  0001 C CNN
 F 3 "" H 9100 5750 60  0000 C CNN
 	1    9100 5750
